File: projet R/projet/projet.kicad_sch (KiCad schematic)
At the start: 0 parts

Commit message: Update KiCad schematics
Other:
- sheet Actionneurs ports: added ENCOD_A1, ENCOD_A2, ENCOD_B1, ENCOD_B2; removed PHASE_A1, PHASE_A2, PHASE_B1, PHASE_B2
- sheet STM32 ports: added BORDER_3, BORDER_4, ENCOD_A1, ENCOD_A2, ENCOD_B1, ENCOD_B2, LIDAR_M_CTR; removed LIDAR_DEV_EN, LIDAR_M_EN, LIDAR_M_SCTR, LIDAR_RX, PHASE_A1, PHASE_A2, PHASE_B1, PHASE_B2
- sheet Sensors ports: added BORDER_3, BORDER_4, LIDAR_M_CTR; removed LIDAR_DEV_EN, LIDAR_M_EN, LIDAR_M_SCTR, LIDAR_RX
Changed lines of the file:
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@@
+	(wire
+		(pts
+			(xy 100.33 80.01) (xy 123.19 80.01)
+		)
+		(stroke
+			(width 0)
+			(type default)
+		)
+	)
 	(wire
 		(pts
@@
 	(wire
 		(pts
-			(xy 172.72 115.57) (xy 193.04 115.57)
-		)
-		(stroke
-			(width 0)
-			(type default)
-		)
-	)
-	(wire
-		(pts
-			(xy 100.33 92.71) (xy 123.19 92.71)
-		)
-		(stroke
-			(width 0)
-			(type default)
-		)
-	)
-	(wire
-		(pts
-			(xy 100.33 95.25) (xy 123.19 95.25)
+			(xy 172.72 96.52) (xy 193.04 96.52)
 		)
 		(stroke
@@
 	(wire
 		(pts
-			(xy 100.33 90.17) (xy 123.19 90.17)
+			(xy 172.72 92.71) (xy 193.04 92.71)
+		)
+		(stroke
+			(width 0)
+			(type default)
+		)
+	)
+	(wire
+		(pts
+			(xy 172.72 88.9) (xy 193.04 88.9)
 		)
 		(stroke
@@
 	(wire
 		(pts
-			(xy 172.72 118.11) (xy 193.04 118.11)
-		)
-		(stroke
-			(width 0)
-			(type default)
-		)
-	)
-	(wire
-		(pts
-			(xy 100.33 87.63) (xy 123.19 87.63)
-		)
-		(stroke
-			(width 0)
-			(type default)
-		)
-	)
-	(wire
-		(pts
-			(xy 172.72 110.49) (xy 193.04 110.49)
-		)
-		(stroke
-			(width 0)
-			(type default)
-		)
-	)
-	(wire
-		(pts
-			(xy 172.72 113.03) (xy 193.04 113.03)
+			(xy 172.72 100.33) (xy 193.04 100.33)
+		)
+		(stroke
+			(width 0)
+			(type default)
+		)
+	)
+	(wire
+		(pts
+			(xy 100.33 93.98) (xy 123.19 93.98)
+		)
+		(stroke
+			(width 0)
+			(type default)
+		)
+	)
+	(wire
+		(pts
+			(xy 100.33 77.47) (xy 123.19 77.47)
 		)
 		(stroke
@@
 			)
 		)
-		(pin "PHASE_A1" input
-			(at 193.04 110.49 180)
-			(effects
-				(font
-					(size 1.27 1.27)
-				)
-				(justify left)
-			)
-		)
-		(pin "PHASE_A2" input
-			(at 193.04 115.57 180)
-			(effects
-				(font
-					(size 1.27 1.27)
-				)
-				(justify left)
-			)
-		)
-		(pin "PHASE_B1" input
-			(at 193.04 113.03 180)
-			(effects
-				(font
-					(size 1.27 1.27)
-				)
-				(justify left)
-			)
-		)
-		(pin "PHASE_B2" input
-			(at 193.04 118.11 180)
-			(effects
-				(font
-					(size 1.27 1.27)
-				)
-				(justify left)
-			)
-		)
 		(pin "REV1" input
 			(at 193.04 123.19 180)
@@
 		(pin "REV2" input
 			(at 193.04 125.73 180)
+			(effects
+				(font
+					(size 1.27 1.27)
+				)
+				(justify left)
+			)
+		)
+		(pin "ENCOD_A1" input
+			(at 193.04 88.9 180)
+			(effects
+				(font
+					(size 1.27 1.27)
+				)
+				(justify left)
+			)
+		)
+		(pin "ENCOD_A2" input
+			(at 193.04 92.71 180)
+			(effects
+				(font
+					(size 1.27 1.27)
+				)
+				(justify left)
+			)
+		)
+		(pin "ENCOD_B1" input
+			(at 193.04 96.52 180)
+			(effects
+				(font
+					(size 1.27 1.27)
+				)
+				(justify left)
+			)
+		)
+		(pin "ENCOD_B2" input
+			(at 193.04 100.33 180)
 			(effects
 				(font
@@
 			)
 		)
-		(pin "BORDER_1" output
-			(at 123.19 72.39 180)
-			(effects
-				(font
-					(size 1.27 1.27)
-				)
-				(justify left)
-			)
-		)
-		(pin "BORDER_2" output
-			(at 123.19 74.93 180)
-			(effects
-				(font
-					(size 1.27 1.27)
-				)
-				(justify left)
-			)
-		)
 		(pin "FWD2" output
 			(at 172.72 130.81 0)
@@
 			)
 		)
-		(pin "LIDAR_DEV_EN" output
-			(at 123.19 87.63 180)
-			(effects
-				(font
-					(size 1.27 1.27)
-				)
-				(justify left)
-			)
-		)
-		(pin "LIDAR_M_EN" output
-			(at 123.19 90.17 180)
-			(effects
-				(font
-					(size 1.27 1.27)
-				)
-				(justify left)
-			)
-		)
-		(pin "LIDAR_M_SCTR" output
-			(at 123.19 92.71 180)
-			(effects
-				(font
-					(size 1.27 1.27)
-				)
-				(justify left)
-			)
-		)
-		(pin "LIDAR_RX" input
-			(at 123.19 95.25 180)
-			(effects
-				(font
-					(size 1.27 1.27)
-				)
-				(justify left)
-			)
-		)
 		(pin "LIDAR_TX" output
 			(at 123.19 97.79 180)
@@
 			)
 		)
-		(pin "PHASE_A1" input
-			(at 172.72 110.49 0)
-			(effects
-				(font
-					(size 1.27 1.27)
-				)
-				(justify right)
-			)
-		)
-		(pin "PHASE_B1" input
-			(at 172.72 113.03 0)
-			(effects
-				(font
-					(size 1.27 1.27)
-				)
-				(justify right)
-			)
-		)
-		(pin "PHASE_B2" input
-			(at 172.72 118.11 0)
-			(effects
-				(font
-					(size 1.27 1.27)
-				)
-				(justify right)
-			)
-		)
 		(pin "REV1" output
 			(at 172.72 123.19 0)
@@
 			)
 		)
-		(pin "PHASE_A2" input
-			(at 172.72 115.57 0)
-			(effects
-				(font
-					(size 1.27 1.27)
-				)
-				(justify right)
+		(pin "LIDAR_M_CTR" input
+			(at 123.19 93.98 180)
+			(effects
+				(font
+					(size 1.27 1.27)
+				)
+				(justify left)
+			)
+		)
+		(pin "ENCOD_A1" input
+			(at 172.72 88.9 0)
+			(effects
+				(font
+					(size 1.27 1.27)
+				)
+				(justify right)
+			)
+		)
+		(pin "ENCOD_A2" input
+			(at 172.72 92.71 0)
+			(effects
+				(font
+					(size 1.27 1.27)
+				)
+				(justify right)
+			)
+		)
+		(pin "ENCOD_B1" input
+			(at 172.72 96.52 0)
+			(effects
+				(font
+					(size 1.27 1.27)
+				)
+				(justify right)
+			)
+		)
+		(pin "ENCOD_B2" input
+			(at 172.72 100.33 0)
+			(effects
+				(font
+					(size 1.27 1.27)
+				)
+				(justify right)
+			)
+		)
+		(pin "BORDER_1" input
+			(at 123.19 72.39 180)
+			(effects
+				(font
+					(size 1.27 1.27)
+				)
+				(justify left)
+			)
+		)
+		(pin "BORDER_2" input
+			(at 123.19 74.93 180)
+			(effects
+				(font
+					(size 1.27 1.27)
+				)
+				(justify left)
+			)
+		)
+		(pin "BORDER_3" input
+			(at 123.19 77.47 180)
+			(effects
+				(font
+					(size 1.27 1.27)
+				)
+				(justify left)
+			)
+		)
+		(pin "BORDER_4" input
+			(at 123.19 80.01 180)
+			(effects
+				(font
+					(size 1.27 1.27)
+				)
+				(justify left)
 			)
 		)
@@
 			)
 		)
-		(pin "LIDAR_DEV_EN" input
-			(at 100.33 87.63 0)
-			(effects
-				(font
-					(size 1.27 1.27)
-				)
-				(justify right)
-			)
-		)
-		(pin "LIDAR_M_EN" input
-			(at 100.33 90.17 0)
-			(effects
-				(font
-					(size 1.27 1.27)
-				)
-				(justify right)
-			)
-		)
-		(pin "LIDAR_M_SCTR" input
-			(at 100.33 92.71 0)
-			(effects
-				(font
-					(size 1.27 1.27)
-				)
-				(justify right)
-			)
-		)
-		(pin "LIDAR_RX" input
-			(at 100.33 95.25 0)
-			(effects
-				(font
-					(size 1.27 1.27)
-				)
-				(justify right)
-			)
-		)
 		(pin "LIDAR_TX" output
 			(at 100.33 97.79 0)
@@
 			(effects
 				(font
+					(size 1.27 1.27)
+				)
+				(justify right)
+			)
+		)
+		(pin "LIDAR_M_CTR" input
+			(at 100.33 93.98 0)
+			(effects
+				(font
+					(size 1.27 1.27)
+				)
+				(justify right)
+			)
+		)
+		(pin "BORDER_3" output
+			(at 100.33 77.47 0)
+			(effects
+				(font
+					(size 1.27 1.27)
+				)
+				(justify right)
+			)
+		)
+		(pin "BORDER_4" output
+			(at 100.33 80.01 0)
+			(effects
+				(font

Commit message: Updated project
Other:
- sheet STM32 ports: added BLE_RX, BLE_TX; removed none
- sheet Sensors ports: added BLE_RX, BLE_TX; removed none
Changed lines of the file:
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@@
+	(wire
+		(pts
+			(xy 100.33 118.11) (xy 123.19 118.11)
+		)
+		(stroke
+			(width 0)
+			(type default)
+		)
+	)
 	(wire
 		(pts
@@
 		(pts
 			(xy 100.33 74.93) (xy 123.19 74.93)
+		)
+		(stroke
+			(width 0)
+			(type default)
+		)
+	)
+	(wire
+		(pts
+			(xy 100.33 115.57) (xy 123.19 115.57)
 		)
 		(stroke
@@
 			)
 		)
+		(pin "BLE_RX" input
+			(at 123.19 115.57 180)
+			(effects
+				(font
+					(size 1.27 1.27)
+				)
+				(justify left)
+			)
+		)
+		(pin "BLE_TX" input
+			(at 123.19 118.11 180)
+			(effects
+				(font
+					(size 1.27 1.27)
+				)
+				(justify left)
+			)
+		)
 		(instances
 			(project "projet"
@@
 			(effects
 				(font
+					(size 1.27 1.27)
+				)
+				(justify right)
+			)
+		)
+		(pin "BLE_RX" input
+			(at 100.33 115.57 0)
+			(effects
+				(font
+					(size 1.27 1.27)
+				)
+				(justify right)
+			)
+		)
+		(pin "BLE_TX" input
+			(at 100.33 118.11 0)
+			(effects
+				(font
