File: projet R/projet/Actionneurs.kicad_sch (KiCad schematic)
At the start: 16 parts, among them J3 Conn_01x06, J5 Conn_01x06, U2 ZXBM5210-SP, U3 ZXBM5210-SP

Commit message: Update KiCad schematics
Connections:
- net MOTEUR1+: no longer J3.6 (Pin_6)
- net MOTEUR1-: no longer J3.1 (Pin_1)
- net PHASE_A1 renamed ENCOD_A1
- net PHASE_A2 renamed ENCOD_A2
- net PHASE_B1 renamed ENCOD_B1
- net PHASE_B2 renamed ENCOD_B2
Changed lines of the file:
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@@
+	(wire
+		(pts
+			(xy 173.99 105.41) (xy 184.15 105.41)
+		)
+		(stroke
+			(width 0)
+			(type default)
+		)
+	)
 	(wire
 		(pts
@@
 	(wire
 		(pts
+			(xy 173.99 92.71) (xy 184.15 92.71)
+		)
+		(stroke
+			(width 0)
+			(type default)
+		)
+	)
+	(wire
+		(pts
 			(xy 68.58 106.68) (xy 72.39 106.68)
 		)
@@
 	(wire
 		(pts
-			(xy 180.34 92.71) (xy 184.15 92.71)
-		)
-		(stroke
-			(width 0)
-			(type default)
-		)
-	)
-	(wire
-		(pts
 			(xy 92.71 128.27) (xy 96.52 128.27)
 		)
@@
 		(pts
 			(xy 69.85 40.64) (xy 69.85 57.15)
-		)
-		(stroke
-			(width 0)
-			(type default)
-		)
-	)
-	(wire
-		(pts
-			(xy 180.34 105.41) (xy 184.15 105.41)
 		)
 		(stroke
@@
 	)
 	(label "MOTEUR1-"
+		(at 170.18 66.04 180)
+		(effects
+			(font
+				(size 1.27 1.27)
+			)
+			(justify right bottom)
+		)
+	)
+	(label "MOTEUR1-"
 		(at 115.57 62.23 0)
 		(effects
@@
 		)
 	)
-	(global_label "MOTEUR2+"
-		(shape input)
-		(at 180.34 105.41 180)
-		(fields_autoplaced yes)
+	(label "MOTEUR2-"
+		(at 173.99 92.71 180)
+		(effects
+			(font
+				(size 1.27 1.27)
+			)
+			(justify right bottom)
+		)
+	)
+	(label "MOTEUR1+"
+		(at 171.45 80.01 180)
+		(effects
+			(font
+				(size 1.27 1.27)
+			)
+			(justify right bottom)
+		)
+	)
+	(label "MOTEUR2+"
+		(at 173.99 105.41 180)
+		(effects
+			(font
+				(size 1.27 1.27)
+			)
+			(justify right bottom)
+		)
+	)
+	(hierarchical_label "FWD1"
+		(shape input)
+		(at 66.04 59.69 180)
 		(effects
 			(font
@@
 			(justify right)
 		)
-		(property "Intersheetrefs" "${INTERSHEET_REFS}"
-			(at 167.0739 105.41 0)
-			(effects
-				(font
-					(size 1.27 1.27)
-				)
-				(justify right)
-				(hide yes)
-			)
-		)
-	)
-	(global_label "MOTEUR1-"
-		(shape input)
-		(at 180.34 66.04 180)
-		(fields_autoplaced yes)
+	)
+	(hierarchical_label "ENCOD_B1"
+		(shape input)
+		(at 180.34 73.66 180)
 		(effects
 			(font
@@
 			(justify right)
 		)
-		(property "Intersheetrefs" "${INTERSHEET_REFS}"
-			(at 167.0739 66.04 0)
-			(effects
-				(font
-					(size 1.27 1.27)
-				)
-				(justify right)
-				(hide yes)
-			)
-		)
-	)
-	(global_label "MOTEUR2-"
-		(shape input)
-		(at 180.34 92.71 180)
-		(fields_autoplaced yes)
+	)
+	(hierarchical_label "ENCOD_B2"
+		(shape input)
+		(at 180.34 100.33 180)
 		(effects
 			(font
@@
 			(justify right)
 		)
-		(property "Intersheetrefs" "${INTERSHEET_REFS}"
-			(at 167.0739 92.71 0)
-			(effects
-				(font
-					(size 1.27 1.27)
-				)
-				(justify right)
-				(hide yes)
-			)
-		)
-	)
-	(global_label "MOTEUR1+"
-		(shape input)
-		(at 180.34 78.74 180)
-		(fields_autoplaced yes)
+	)
+	(hierarchical_label "FWD2"
+		(shape input)
+		(at 64.77 125.73 180)
 		(effects
 			(font
@@
 			(justify right)
 		)
-		(property "Intersheetrefs" "${INTERSHEET_REFS}"
-			(at 167.0739 78.74 0)
-			(effects
-				(font
-					(size 1.27 1.27)
-				)
-				(justify right)
-				(hide yes)
-			)
-		)
-	)
-	(hierarchical_label "FWD1"
-		(shape input)
-		(at 66.04 59.69 180)
+	)
+	(hierarchical_label "ENCOD_A1"
+		(shape input)
+		(at 180.34 71.12 180)
 		(effects
 			(font
@@
 		)
 	)
-	(hierarchical_label "PHASE_B1"
-		(shape input)
-		(at 180.34 73.66 180)
+	(hierarchical_label "REV1"
+		(shape input)
+		(at 66.04 62.23 180)
 		(effects
 			(font
@@
 		)
 	)
-	(hierarchical_label "PHASE_B2"
-		(shape input)
-		(at 180.34 100.33 180)
+	(hierarchical_label "REV2"
+		(shape input)
+		(at 64.77 128.27 180)
 		(effects
 			(font
@@
 		)
 	)
-	(hierarchical_label "FWD2"
-		(shape input)
-		(at 64.77 125.73 180)
-		(effects
-			(font
-				(size 1.27 1.27)
-			)
-			(justify right)
-		)
-	)
-	(hierarchical_label "PHASE_A1"
-		(shape input)
-		(at 180.34 71.12 180)
-		(effects
-			(font
-				(size 1.27 1.27)
-			)
-			(justify right)
-		)
-	)
-	(hierarchical_label "REV1"
-		(shape input)
-		(at 66.04 62.23 180)
-		(effects
-			(font
-				(size 1.27 1.27)
-			)
-			(justify right)
-		)
-	)
-	(hierarchical_label "REV2"
-		(shape input)
-		(at 64.77 128.27 180)
-		(effects
-			(font
-				(size 1.27 1.27)
-			)
-			(justify right)
-		)
-	)
-	(hierarchical_label "PHASE_A2"
+	(hierarchical_label "ENCOD_A2"
 		(shape input)
 		(at 180.34 97.79 180)

Commit message: Updated project
Parts:
- C12, C13, C14, C15, C16, C17, C18, C19: footprint (none) -> Capacitor_SMD:C_01005_0402Metric
Changed lines of the file:
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@@
 			)
 		)
-		(property "Footprint" ""
+		(property "Footprint" "Capacitor_SMD:C_01005_0402Metric"
 			(at 96.52 119.38 0)
 			(effects
@@
 			)
 		)
-		(property "Footprint" ""
+		(property "Footprint" "Capacitor_SMD:C_01005_0402Metric"
 			(at 116.84 43.18 0)
 			(effects
@@
 			)
 		)
-		(property "Footprint" ""
+		(property "Footprint" "Capacitor_SMD:C_01005_0402Metric"
 			(at 97.79 64.77 0)
 			(effects
@@
 			)
 		)
-		(property "Footprint" ""
+		(property "Footprint" "Capacitor_SMD:C_01005_0402Metric"
 			(at 106.68 109.22 0)
 			(effects
@@
 			)
 		)
-		(property "Footprint" ""
+		(property "Footprint" "Capacitor_SMD:C_01005_0402Metric"
 			(at 97.79 53.34 0)
 			(effects
@@
 			)
 		)
-		(property "Footprint" ""
+		(property "Footprint" "Capacitor_SMD:C_01005_0402Metric"
 			(at 107.95 43.18 0)
 			(effects
@@
 			)
 		)
-		(property "Footprint" ""
+		(property "Footprint" "Capacitor_SMD:C_01005_0402Metric"
 			(at 96.52 130.81 0)
 			(effects
@@
 			)
 		)
-		(property "Footprint" ""
+		(property "Footprint" "Capacitor_SMD:C_01005_0402Metric"
 			(at 115.57 109.22 0)
 			(effects

Commit message: Updated project
Parts:
- C12, C13, C14, C15, C16, C17, C18, C19: footprint Capacitor_SMD:C_01005_0402Metric -> Capacitor_SMD:C_0402_1005Metric
Changed lines of the file:
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@@
 			)
 		)
-		(property "Footprint" "Capacitor_SMD:C_01005_0402Metric"
+		(property "Footprint" "Capacitor_SMD:C_0402_1005Metric"
 			(at 96.52 119.38 0)
 			(effects
@@
 			)
 		)
-		(property "Footprint" "Capacitor_SMD:C_01005_0402Metric"
+		(property "Footprint" "Capacitor_SMD:C_0402_1005Metric"
 			(at 116.84 43.18 0)
 			(effects
@@
 			)
 		)
-		(property "Footprint" "Capacitor_SMD:C_01005_0402Metric"
+		(property "Footprint" "Capacitor_SMD:C_0402_1005Metric"
 			(at 97.79 64.77 0)
 			(effects
@@
 			)
 		)
-		(property "Footprint" "Capacitor_SMD:C_01005_0402Metric"
+		(property "Footprint" "Capacitor_SMD:C_0402_1005Metric"
 			(at 106.68 109.22 0)
 			(effects
@@
 			)
 		)
-		(property "Footprint" "Capacitor_SMD:C_01005_0402Metric"
+		(property "Footprint" "Capacitor_SMD:C_0402_1005Metric"
 			(at 97.79 53.34 0)
 			(effects
@@
 			)
 		)
-		(property "Footprint" "Capacitor_SMD:C_01005_0402Metric"
+		(property "Footprint" "Capacitor_SMD:C_0402_1005Metric"
 			(at 107.95 43.18 0)
 			(effects
@@
 			)
 		)
-		(property "Footprint" "Capacitor_SMD:C_01005_0402Metric"
+		(property "Footprint" "Capacitor_SMD:C_0402_1005Metric"
 			(at 96.52 130.81 0)
 			(effects
@@
 			)
 		)
-		(property "Footprint" "Capacitor_SMD:C_01005_0402Metric"
+		(property "Footprint" "Capacitor_SMD:C_0402_1005Metric"
 			(at 115.57 109.22 0)
 			(effects
