File: projet R/projet/Alimentation.kicad_sch (KiCad schematic)
At the start: 27 parts, among them IC1 MP1475DJ-LF-P, J2 Screw_Terminal_01x02, SW1 ON/OFF

Commit message: Updated project
Parts:
- 3V3, TP7: footprint (none) -> TestPoint:TestPoint_Pad_D1.0mm
- C23, C24, C25, C26, C27, C28, C29, C30: footprint (none) -> Capacitor_SMD:C_01005_0402Metric
- D2_PWR_5V1: renamed from D2_PWR_5V; footprint (none) -> LED_SMD:LED_0603_1608Metric
- D3_PWR_3V1: renamed from D3_PWR_3V; footprint (none) -> LED_SMD:LED_0603_1608Metric
- J2: footprint (none) -> Connector_JST:JST_XH_S2B-XH-A_1x02_P2.50mm_Horizontal
- R10, R11, R12, R13, R14, R15: footprint (none) -> Resistor_SMD:R_0402_1005Metric
- R2: value 1k -> 240; footprint (none) -> Resistor_SMD:R_0402_1005Metric
- R3: value 1k -> 160; footprint (none) -> Resistor_SMD:R_0402_1005Metric
- R4: value 1k -> 100; footprint (none) -> Resistor_SMD:R_0402_1005Metric
- renumbered D1_PWR_BATT to D1_PWR_BATT1
Connections:
- net +7.2V: no longer names the net of J2.1 (Pin_1), SW1.3 (A)
Other:
- moved on the sheet: J2
Changed lines of the file:
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@@
 	(wire
 		(pts
-			(xy 36.83 40.64) (xy 36.83 41.91)
-		)
-		(stroke
-			(width 0)
-			(type default)
-		)
-	)
-	(wire
-		(pts
 			(xy 33.02 82.55) (xy 38.1 82.55)
 		)
@@
 	(wire
 		(pts
+			(xy 48.26 48.26) (xy 57.15 48.26)
+		)
+		(stroke
+			(width 0)
+			(type default)
+		)
+	)
+	(wire
+		(pts
 			(xy 195.58 60.96) (xy 195.58 63.5)
 		)
@@
 	(wire
 		(pts
-			(xy 67.31 45.72) (xy 69.85 45.72)
+			(xy 48.26 43.18) (xy 48.26 45.72)
 		)
 		(stroke
@@
 		)
 	)
-	(global_label "+7.2V"
-		(shape input)
-		(at 57.15 48.26 180)
-		(fields_autoplaced yes)
-		(effects
-			(font
-				(size 1.27 1.27)
-			)
-			(justify right)
-		)
-		(property "Intersheetrefs" "${INTERSHEET_REFS}"
-			(at 48.48 48.26 0)
-			(effects
-				(font
-					(size 1.27 1.27)
-				)
-				(justify right)
-				(hide yes)
-			)
-		)
-	)
-	(global_label "+7.2V"
-		(shape input)
-		(at 36.83 38.1 180)
-		(fields_autoplaced yes)
-		(effects
-			(font
-				(size 1.27 1.27)
-			)
-			(justify right)
+	(wire
+		(pts
+			(xy 67.31 45.72) (xy 69.85 45.72)
 		)
-		(property "Intersheetrefs" "${INTERSHEET_REFS}"
-			(at 28.16 38.1 0)
-			(effects
-				(font
-					(size 1.27 1.27)
-				)
-				(justify right)
-				(hide yes)
-			)
+		(stroke
+			(width 0)
+			(type default)
 		)
 	)
@@
 		(dnp no)
 		(fields_autoplaced yes)
-		(property "Reference" "D3_PWR_3V"
+		(property "Reference" "D3_PWR_3V1"
 			(at 43.4975 86.36 0)
 			(effects
@@
 			)
 		)
-		(property "Footprint" ""
+		(property "Footprint" "LED_SMD:LED_0603_1608Metric"
 			(at 41.91 93.98 0)
 			(effects
@@
 			(project ""
 				(path "/b2330267-3262-4d12-877e-36612b3f2d84/027c0f16-9d10-4b80-857c-f21dafef43b8"
-					(reference "D3_PWR_3V")
+					(reference "D3_PWR_3V1")
 					(unit 1)
 				)
@@
 			)
 		)
-		(property "Footprint" ""
+		(property "Footprint" "Resistor_SMD:R_0402_1005Metric"
 			(at 115.57 64.77 0)
 			(effects
@@
 			)
 		)
-		(property "Footprint" ""
+		(property "Footprint" "Capacitor_SMD:C_01005_0402Metric"
 			(at 91.44 62.23 0)
 			(effects
@@
 			)
 		)
-		(property "Value" "1k"
+		(property "Value" "240"
 			(at 53.34 71.12 90)
 			(effects
@@
 			)
 		)
-		(property "Footprint" ""
+		(property "Footprint" "Resistor_SMD:R_0402_1005Metric"
 			(at 53.34 73.66 0)
 			(effects
@@
 			)
 		)
-		(property "Footprint" ""
+		(property "Footprint" "Resistor_SMD:R_0402_1005Metric"
 			(at 171.45 74.93 0)
 			(effects
@@
 			)
 		)
-		(property "Footprint" ""
+		(property "Footprint" "TestPoint:TestPoint_Pad_D1.0mm"
 			(at 273.05 59.69 0)
 			(effects
@@
 	(symbol
 		(lib_id "Connector:Screw_Terminal_01x02")
-		(at 41.91 38.1 0)
+		(at 43.18 48.26 180)
 		(unit 1)
 		(exclude_from_sim no)
@@
 		(fields_autoplaced yes)
 		(property "Reference" "J2"
-			(at 44.45 38.0999 0)
+			(at 43.18 41.91 0)
 			(effects
 				(font
 					(size 1.27 1.27)
 				)
-				(justify left)
 			)
 		)
 		(property "Value" "Screw_Terminal_01x02"
-			(at 44.45 40.6399 0)
+			(at 40.64 45.7201 0)
 			(effects
 				(font
@@
 			)
 		)
-		(property "Footprint" ""
-			(at 41.91 38.1 0)
+		(property "Footprint" "Connector_JST:JST_XH_S2B-XH-A_1x02_P2.50mm_Horizontal"
+			(at 43.18 48.26 0)
 			(effects
 				(font
@@
 		)
 		(property "Datasheet" "~"
-			(at 41.91 38.1 0)
+			(at 43.18 48.26 0)
 			(effects
 				(font
@@
 		)
 		(property "Description" "Generic screw terminal, single row, 01x02, script generated (kicad-library-utils/schlib/autogen/connector/)"
-			(at 41.91 38.1 0)
+			(at 43.18 48.26 0)
 			(effects
 				(font
@@
 		(dnp no)
 		(fields_autoplaced yes)
-		(property "Reference" "D2_PWR_5V"
+		(property "Reference" "D2_PWR_5V1"
 			(at 43.4975 74.93 0)
 			(effects
@@
 			)
 		)
-		(property "Footprint" ""
+		(property "Footprint" "LED_SMD:LED_0603_1608Metric"
 			(at 41.91 82.55 0)
 			(effects
@@
 			(project ""
 				(path "/b2330267-3262-4d12-877e-36612b3f2d84/027c0f16-9d10-4b80-857c-f21dafef43b8"
-					(reference "D2_PWR_5V")
+					(reference "D2_PWR_5V1")
 					(unit 1)
 				)
@@
 			)
 		)
-		(property "Footprint" ""
+		(property "Footprint" "TestPoint:TestPoint_Pad_D1.0mm"
 			(at 208.28 62.23 0)
 			(effects
@@
 			)
 		)
-		(property "Footprint" ""
+		(property "Footprint" "Capacitor_SMD:C_01005_0402Metric"
 			(at 82.55 62.23 0)
 			(effects
@@
 			)
 		)
-		(property "Footprint" ""
+		(property "Footprint" "Resistor_SMD:R_0402_1005Metric"
 			(at 100.33 62.23 0)
 			(effects
@@
 			)
 		)
-		(property "Footprint" ""
+		(property "Footprint" "Capacitor_SMD:C_01005_0402Metric"
 			(at 162.56 60.96 0)
 			(effects
@@
 			)
 		)
-		(property "Footprint" ""
+		(property "Footprint" "Resistor_SMD:R_0402_1005Metric"
 			(at 158.75 58.42 0)
 			(effects
@@
 			)
 		)
-		(property "Footprint" ""
+		(property "Footprint" "Resistor_SMD:R_0402_1005Metric"
 			(at 165.1 88.9 0)
 			(effects
@@
 			)
 		)
-		(property "Value" "1k"
+		(property "Value" "100"
 			(at 53.34 91.44 90)
 			(effects
@@
 			)
 		)
-		(property "Footprint" ""
+		(property "Footprint" "Resistor_SMD:R_0402_1005Metric"
 			(at 53.34 93.98 0)
 			(effects
@@
 			)
 		)
-		(property "Footprint" ""
+		(property "Footprint" "Capacitor_SMD:C_01005_0402Metric"
 			(at 261.62 62.23 0)
 			(effects
@@
 			)
 		)
-		(property "Footprint" ""
+		(property "Footprint" "Capacitor_SMD:C_01005_0402Metric"
 			(at 184.15 66.04 0)
 			(effects
@@
 		(dnp no)
 		(fields_autoplaced yes)
-		(property "Reference" "D1_PWR_BATT"
+		(property "Reference" "D1_PWR_BATT1"
 			(at 43.4975 66.04 0)
 			(effects
@@
 			(project ""
 				(path "/b2330267-3262-4d12-877e-36612b3f2d84/027c0f16-9d10-4b80-857c-f21dafef43b8"
-					(reference "D1_PWR_BATT")
+					(reference "D1_PWR_BATT1")
 					(unit 1)
 				)
@@
 			)
 		)
-		(property "Footprint" ""
+		(property "Footprint" "Resistor_SMD:R_0402_1005Metric"
 			(at 160.02 74.93 0)
 			(effects
@@
 	(symbol
 		(lib_id "power:GND")
-		(at 36.83 41.91 0)
+		(at 48.26 43.18 180)
 		(unit 1)
 		(exclude_from_sim no)
@@
 		(fields_autoplaced yes)
 		(property "Reference" "#PWR015"
-			(at 36.83 48.26 0)
+			(at 48.26 36.83 0)
 			(effects
 				(font
@@
 		)
 		(property "Value" "GND"
-			(at 36.83 46.99 0)
+			(at 50.8 41.9099 0)
 			(effects
 				(font
 					(size 1.27 1.27)
 				)
+				(justify right)
 			)
 		)
 		(property "Footprint" ""
-			(at 36.83 41.91 0)
+			(at 48.26 43.18 0)
 			(effects
 				(font
@@
 		)
 		(property "Datasheet" ""
-			(at 36.83 41.91 0)
+			(at 48.26 43.18 0)
 			(effects
 				(font
@@
 		)
 		(property "Description" "Power symbol creates a global label with name \"GND\" , ground"
-			(at 36.83 41.91 0)
+			(at 48.26 43.18 0)
 			(effects
 				(font
@@
 		)
 		(instances
-			(project ""
+			(project "projet"
 				(path "/b2330267-3262-4d12-877e-36612b3f2d84/027c0f16-9d10-4b80-857c-f21dafef43b8"
 					(reference "#PWR015")
@@
 			)
 		)
-		(property "Value" "1k"
+		(property "Value" "160"
 			(at 53.34 80.01 90)
 			(effects
@@
 			)
 		)
-		(property "Footprint" ""
+		(property "Footprint" "Resistor_SMD:R_0402_1005Metric"
 			(at 53.34 82.55 0)
 			(effects
@@
 			)
 		)
-		(property "Footprint" ""
+		(property "Footprint" "Capacitor_SMD:C_01005_0402Metric"
 			(at 171.45 83.82 0)
 			(effects
@@
 			)
 		)
-		(property "Footprint" ""
+		(property "Footprint" "Capacitor_SMD:C_01005_0402Metric"
 			(at 195.58 66.04 0)
 			(effects
@@
 			)
 		)
-		(property "Footprint" ""
+		(property "Footprint" "Capacitor_SMD:C_01005_0402Metric"
 			(at 107.95 64.77 0)
 			(effects

Commit message: Updated project
Parts:
- added C4: 0.47u, Capacitor_SMD:C_01005_0402Metric, symbol Device:C_Small
- C23, C24, C25, C26, C27, C28, C29, C30: footprint Capacitor_SMD:C_01005_0402Metric -> Capacitor_SMD:C_0402_1005Metric
- R14: value R_Small -> 16k
- R2: value 240 -> 5k5
- R3: value 160 -> 3k3
- R4: value 100 -> 1k6
Connections:
- net +5V: now also C4.1
- net GND: now also C4.2
Other:
- moved on the sheet: C24, C25
Changed lines of the file:
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@@
 	)
 	(junction
+		(at 218.44 62.23)
+		(diameter 0)
+		(color 0 0 0 0)
+	)
+	(junction
 		(at 195.58 63.5)
 		(diameter 0)
@@
 	)
 	(junction
-		(at 82.55 59.69)
+		(at 82.55 58.42)
 		(diameter 0)
 		(color 0 0 0 0)
@@
 	)
 	(junction
-		(at 91.44 59.69)
+		(at 91.44 58.42)
 		(diameter 0)
 		(color 0 0 0 0)
@@
 	)
 	(junction
-		(at 82.55 64.77)
+		(at 82.55 63.5)
 		(diameter 0)
 		(color 0 0 0 0)
@@
 	(wire
 		(pts
-			(xy 82.55 64.77) (xy 82.55 67.31)
+			(xy 82.55 63.5) (xy 82.55 66.04)
 		)
 		(stroke
@@
 	(wire
 		(pts
-			(xy 227.33 62.23) (xy 218.44 62.23)
+			(xy 218.44 62.23) (xy 227.33 62.23)
 		)
 		(stroke
@@
 	(wire
 		(pts
+			(xy 218.44 66.04) (xy 218.44 62.23)
+		)
+		(stroke
+			(width 0)
+			(type default)
+		)
+	)
+	(wire
+		(pts
 			(xy 55.88 82.55) (xy 60.96 82.55)
 		)
@@
 	(wire
 		(pts
-			(xy 82.55 59.69) (xy 91.44 59.69)
+			(xy 82.55 58.42) (xy 91.44 58.42)
 		)
 		(stroke
@@
 	(wire
 		(pts
-			(xy 82.55 64.77) (xy 91.44 64.77)
+			(xy 82.55 63.5) (xy 91.44 63.5)
 		)
 		(stroke
@@
 	(wire
 		(pts
-			(xy 82.55 53.34) (xy 82.55 59.69)
+			(xy 82.55 52.07) (xy 82.55 58.42)
 		)
 		(stroke
@@
 	(wire
 		(pts
-			(xy 91.44 58.42) (xy 91.44 59.69)
-		)
-		(stroke
-			(width 0)
-			(type default)
-		)
-	)
-	(wire
-		(pts
 			(xy 48.26 43.18) (xy 48.26 45.72)
 		)
@@
 	)
 	(symbol
+		(lib_id "Device:C_Small")
+		(at 218.44 68.58 0)
+		(unit 1)
+		(exclude_from_sim no)
+		(in_bom yes)
+		(on_board yes)
+		(dnp no)
+		(fields_autoplaced yes)
+		(property "Reference" "C4"
+			(at 220.98 67.3162 0)
+			(effects
+				(font
+					(size 1.27 1.27)
+				)
+				(justify left)
+			)
+		)
+		(property "Value" "0.47u"
+			(at 220.98 69.8562 0)
+			(effects
+				(font
+					(size 1.27 1.27)
+				)
+				(justify left)
+			)
+		)
+		(property "Footprint" "Capacitor_SMD:C_01005_0402Metric"
+			(at 218.44 68.58 0)
+			(effects
+				(font
+					(size 1.27 1.27)
+				)
+				(hide yes)
+			)
+		)
+		(property "Datasheet" "~"
+			(at 218.44 68.58 0)
+			(effects
+				(font
+					(size 1.27 1.27)
+				)
+				(hide yes)
+			)
+		)
+		(property "Description" "Unpolarized capacitor, small symbol"
+			(at 218.44 68.58 0)
+			(effects
+				(font
+					(size 1.27 1.27)
+				)
+				(hide yes)
+			)
+		)
+		(pin "1"
+		)
+		(pin "2"
+		)
+		(instances
+			(project "projet"
+				(path "/b2330267-3262-4d12-877e-36612b3f2d84/027c0f16-9d10-4b80-857c-f21dafef43b8"
+					(reference "C4")
+					(unit 1)
+				)
+			)
+		)
+	)
+	(symbol
 		(lib_id "Switch:SW_Nidec_CAS-120A1")
 		(at 62.23 45.72 180)
@@
 	(symbol
 		(lib_id "Device:C_Small")
-		(at 91.44 62.23 0)
+		(at 91.44 60.96 0)
 		(unit 1)
 		(exclude_from_sim no)
@@
 		(fields_autoplaced yes)
 		(property "Reference" "C25"
-			(at 93.98 60.9662 0)
+			(at 93.98 59.6962 0)
 			(effects
 				(font
@@
 		)
 		(property "Value" "100nF"
-			(at 93.98 63.5062 0)
+			(at 93.98 62.2362 0)
 			(effects
 				(font
@@
 			)
 		)
-		(property "Footprint" "Capacitor_SMD:C_01005_0402Metric"
-			(at 91.44 62.23 0)
+		(property "Footprint" "Capacitor_SMD:C_0402_1005Metric"
+			(at 91.44 60.96 0)
 			(effects
 				(font
@@
 		)
 		(property "Datasheet" "~"
-			(at 91.44 62.23 0)
+			(at 91.44 60.96 0)
 			(effects
 				(font
@@
 		)
 		(property "Description" "Unpolarized capacitor, small symbol"
-			(at 91.44 62.23 0)
+			(at 91.44 60.96 0)
 			(effects
 				(font
@@
 			)
 		)
-		(property "Value" "240"
+		(property "Value" "5k5"
 			(at 53.34 71.12 90)
 			(effects
@@
 	(symbol
 		(lib_id "Device:C_Small")
-		(at 82.55 62.23 0)
+		(at 82.55 60.96 0)
 		(unit 1)
 		(exclude_from_sim no)
@@
 		(fields_autoplaced yes)
 		(property "Reference" "C24"
-			(at 85.09 60.9662 0)
+			(at 85.09 59.6962 0)
 			(effects
 				(font
@@
 		)
 		(property "Value" "22uF"
-			(at 85.09 63.5062 0)
+			(at 85.09 62.2362 0)
 			(effects
 				(font
@@
 			)
 		)
-		(property "Footprint" "Capacitor_SMD:C_01005_0402Metric"
-			(at 82.55 62.23 0)
+		(property "Footprint" "Capacitor_SMD:C_0402_1005Metric"
+			(at 82.55 60.96 0)
 			(effects
 				(font
@@
 		)
 		(property "Datasheet" "~"
-			(at 82.55 62.23 0)
+			(at 82.55 60.96 0)
 			(effects
 				(font
@@
 		)
 		(property "Description" "Unpolarized capacitor, small symbol"
-			(at 82.55 62.23 0)
+			(at 82.55 60.96 0)
 			(effects
 				(font
@@
 	)
 	(symbol
+		(lib_id "power:GND")
+		(at 218.44 71.12 0)
+		(unit 1)
+		(exclude_from_sim no)
+		(in_bom yes)
+		(on_board yes)
+		(dnp no)
+		(fields_autoplaced yes)
+		(property "Reference" "#PWR069"
+			(at 218.44 77.47 0)
+			(effects
+				(font
+					(size 1.27 1.27)
+				)
+				(hide yes)
+			)
+		)
+		(property "Value" "GND"
+			(at 218.44 76.2 0)
+			(effects
+				(font
+					(size 1.27 1.27)
+				)
+			)
+		)
+		(property "Footprint" ""
+			(at 218.44 71.12 0)
+			(effects
+				(font
+					(size 1.27 1.27)
+				)
+				(hide yes)
+			)
+		)
+		(property "Datasheet" ""
+			(at 218.44 71.12 0)
+			(effects
+				(font
+					(size 1.27 1.27)
+				)
+				(hide yes)
+			)
+		)
+		(property "Description" "Power symbol creates a global label with name \"GND\" , ground"
+			(at 218.44 71.12 0)
+			(effects
+				(font
+					(size 1.27 1.27)
+				)
+				(hide yes)
+			)
+		)
+		(pin "1"
+		)
+		(instances
+			(project "projet"
+				(path "/b2330267-3262-4d12-877e-36612b3f2d84/027c0f16-9d10-4b80-857c-f21dafef43b8"
+					(reference "#PWR069")
+					(unit 1)
+				)
+			)
+		)
+	)
+	(symbol
 		(lib_id "power:+BATT")
-		(at 82.55 53.34 0)
+		(at 82.55 52.07 0)
 		(unit 1)
 		(exclude_from_sim no)
@@
 		(fields_autoplaced yes)
 		(property "Reference" "#PWR052"
-			(at 82.55 57.15 0)
+			(at 82.55 55.88 0)
 			(effects
 				(font
@@
 		)
 		(property "Value" "+BATT"
-			(at 82.55 48.26 0)
+			(at 82.55 46.99 0)
 			(effects
 				(font
@@
 		)
 		(property "Footprint" ""
-			(at 82.55 53.34 0)
+			(at 82.55 52.07 0)
 			(effects
 				(font
@@
 		)
 		(property "Datasheet" ""
-			(at 82.55 53.34 0)
+			(at 82.55 52.07 0)
 			(effects
 				(font
@@
 		)
 		(property "Description" "Power symbol creates a global label with name \"+BATT\""
-			(at 82.55 53.34 0)
+			(at 82.55 52.07 0)
 			(effects
 				(font
@@
 			)
 		)
-		(property "Footprint" "Capacitor_SMD:C_01005_0402Metric"
+		(property "Footprint" "Capacitor_SMD:C_0402_1005Metric"
 			(at 162.56 60.96 0)
 			(effects
@@
 			)
 		)
-		(property "Value" "100"
+		(property "Value" "1k6"
 			(at 53.34 91.44 90)
 			(effects
@@
 	(symbol
 		(lib_id "power:GND")
-		(at 82.55 67.31 0)
+		(at 82.55 66.04 0)
 		(unit 1)
 		(exclude_from_sim no)
@@
 		(fields_autoplaced yes)
 		(property "Reference" "#PWR053"
-			(at 82.55 73.66 0)
+			(at 82.55 72.39 0)
 			(effects
 				(font
@@
 		)
 		(property "Value" "GND"
-			(at 82.55 72.39 0)
+			(at 82.55 71.12 0)
 			(effects
 				(font
@@
 		)
 		(property "Footprint" ""
-			(at 82.55 67.31 0)
+			(at 82.55 66.04 0)
 			(effects
 				(font
@@
 		)
 		(property "Datasheet" ""
-			(at 82.55 67.31 0)
+			(at 82.55 66.04 0)
 			(effects
 				(font
@@
 		)
 		(property "Description" "Power symbol creates a global label with name \"GND\" , ground"
-			(at 82.55 67.31 0)
+			(at 82.55 66.04 0)
 			(effects
 				(font
@@
 			)
 		)
-		(property "Footprint" "Capacitor_SMD:C_01005_0402Metric"
+		(property "Footprint" "Capacitor_SMD:C_0402_1005Metric"
 			(at 261.62 62.23 0)
 			(effects
@@
 			)
 		)
-		(property "Footprint" "Capacitor_SMD:C_01005_0402Metric"
+		(property "Footprint" "Capacitor_SMD:C_0402_1005Metric"
 			(at 184.15 66.04 0)
 			(effects
@@
 			)
 		)
-		(property "Value" "R_Small"
+		(property "Value" "16k"
 			(at 160.02 72.39 90)
 			(effects
@@
 			)
 		)
-		(property "Value" "160"
+		(property "Value" "3k3"
 			(at 53.34 80.01 90)
 			(effects
@@
 			)
 		)
-		(property "Footprint" "Capacitor_SMD:C_01005_0402Metric"
+		(property "Footprint" "Capacitor_SMD:C_0402_1005Metric"
 			(at 171.45 83.82 0)
 			(effects
@@
 			)
 		)
-		(property "Footprint" "Capacitor_SMD:C_01005_0402Metric"
+		(property "Footprint" "Capacitor_SMD:C_0402_1005Metric"
 			(at 195.58 66.04 0)
 			(effects
@@
 			)
 		)
-		(property "Footprint" "Capacitor_SMD:C_01005_0402Metric"
+		(property "Footprint" "Capacitor_SMD:C_0402_1005Metric"
 			(at 107.95 64.77 0)
 			(effects
