File: projet R/projet/STM32.kicad_sch (KiCad schematic)
At the start: 25 parts, among them J1 Conn_ST_STDC14, U1 STM32G431CBUx, Y1 Crystal_GND24_Small

Commit message: Update KiCad schematics
Connections:
- net BORDER_1: now also U1.8 (PA0); no longer U1.11 (PA3)
- net BORDER_2: now also U1.9 (PA1); no longer U1.12 (PA4)
- net LIDAR_TX: now also U1.11 (PA3); no longer U1.24 (PB11)
- net REV1: now also U1.46 (PB8); no longer U1.26 (PB13)
- net REV2: now also U1.47 (PB9); no longer U1.27 (PB14)
- net SCL: now also U1.26 (PB13); no longer U1.46 (PB8)
- net SDA: now also U1.27 (PB14); no longer U1.47 (PB9)
- net BORDER_3: now reaches U1.10 (PA2)
- net LIDAR_DEV_EN: no longer names the net of U1.33 (PA11)
- net LIDAR_M_EN: no longer names the net of U1.34 (PA12)
- net LIDAR_M_SCTR renamed LIDAR_M_CTR
- net LIDAR_RX: no longer names the net of U1.22 (PB10)
- net PHASE_A1 renamed ENCOD_A1
- net PHASE_A2 renamed ENCOD_A2
- net PHASE_B1 renamed ENCOD_B1
- net PHASE_B2 renamed ENCOD_B2
- new net BORDER_4: U1.12 (PA4)

Commit message: Updated project
Parts:
- removed C4: 100n, Capacitor_SMD:C_0402_1005Metric, symbol Device:C_Small
- removed L1: L, symbol Device:L
- C22: footprint (none) -> Capacitor_SMD:C_01005_0402Metric
- C3: value 100n -> 4.7uF
- D1, D2, D3: footprint (none) -> LED_SMD:LED_0603_1608Metric
- R7, R8, R9: value 1k -> 100; footprint (none) -> Resistor_SMD:R_0402_1005Metric
Connections:
- net +3.3V: now also C8.2, C9.2, U1.21 (VDDA)
- net BLE_RX: now reaches U1.22 (PB10)
- net BLE_TX: now reaches U1.24 (PB11)

Commit message: Updated project
Parts:
- C22: footprint Capacitor_SMD:C_01005_0402Metric -> Capacitor_SMD:C_0402_1005Metric
- R7, R8, R9: value 100 -> 1k6
Changed lines of the file:
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@@
 			)
 		)
-		(property "Value" "100"
+		(property "Value" "1k6"
 			(at 220.98 52.07 90)
 			(effects
@@
 			)
 		)
-		(property "Value" "100"
+		(property "Value" "1k6"
 			(at 220.98 27.94 90)
 			(effects
@@
 			)
 		)
-		(property "Footprint" "Capacitor_SMD:C_01005_0402Metric"
+		(property "Footprint" "Capacitor_SMD:C_0402_1005Metric"
 			(at 54.61 64.77 0)
 			(effects
@@
 			)
 		)
-		(property "Value" "100"
+		(property "Value" "1k6"
 			(at 220.98 39.37 90)
 			(effects
