File: projet R/projet/Sensors.kicad_sch (KiCad schematic)
At the start: 10 parts, among them J4 BORDER, J6 LIDAR, J7 BORDER, U4 ADXL343

Commit message: Update KiCad schematics
Parts:
- removed J6: LIDAR, Connector_JST:JST_XH_S8B-XH-A_1x08_P2.50mm_Horizontal, symbol Connector_Generic:Conn_01x08
- added C31, C32, C33, C34: 10n, symbol Device:C
- added J10: Conn_01x04, symbol Connector_Generic:Conn_01x04
- added J8, J9: BORDER, Connector_JST:JST_XH_S2B-XH-A_1x02_P2.50mm_Horizontal, symbol Connector_Generic:Conn_01x02
- added R16, R17, R18, R19, R20, R21, R22, R23: 10k, symbol Device:R_Small
Connections:
- net +3.3V: now also R16.1, R18.1, R20.1, R22.1
- net +5V: now also J10.4 (Pin_4)
- net BORDER_1: now also C33.1, R21.2; no longer J4.1 (Pin_1)
- net BORDER_2: now also C31.1, R17.2; no longer J7.1 (Pin_1)
- net GND: now also C31.2, C32.2, C33.2, C34.2, J10.2 (Pin_2), J8.2 (Pin_2), J9.2 (Pin_2)
- net LIDAR_TX: now also J10.3 (Pin_3)
- new net: J7.1 (Pin_1), R16.2, R17.1
- new net: J9.1 (Pin_1), R22.2, R23.1
- new net: J4.1 (Pin_1), R18.2, R19.1
- new net: J8.1 (Pin_1), R20.2, R21.1
- new net BORDER_3: C34.1, R23.2
- new net BORDER_4: C32.1, R19.2
- new net LIDAR_M_CTR: J10.1 (Pin_1)
- no-connect marks 3 -> 2
Other:
- moved on the sheet: J7

Commit message: Updated project
Parts:
- added J11: Conn_01x05, symbol Connector_Generic:Conn_01x05
- C31, C32, C33, C34: footprint (none) -> Capacitor_SMD:C_01005_0402Metric
- J10: footprint (none) -> Connector_JST:JST_XH_S4B-XH-A_1x04_P2.50mm_Horizontal
- R16, R17, R18, R19, R20, R21, R22, R23: footprint (none) -> Resistor_SMD:R_0402_1005Metric
- TP5, TP6: footprint (none) -> TestPoint:TestPoint_Pad_D1.0mm
Connections:
- net +5V: now also J11.5 (Pin_5)
- net GND: now also J11.2 (Pin_2)
- new net BLE_RX: J11.3 (Pin_3)
- new net BLE_TX: J11.4 (Pin_4)
- no-connect marks 2 -> 3
Other:
- note added: "BLEUTOOTH"
- note added: "LIDAR"
- moved on the sheet: J10

Commit message: Updated project
Parts:
- removed J10: Conn_01x04, Connector_JST:JST_XH_S4B-XH-A_1x04_P2.50mm_Horizontal, symbol Connector_Generic:Conn_01x04
- added J6: Conn_01x05, symbol Connector_Generic:Conn_01x05
- C20, C21, C31, C32, C33, C34: footprint Capacitor_SMD:C_01005_0402Metric -> Capacitor_SMD:C_0402_1005Metric
Connections:
- net +5V: now also J6.5 (Pin_5)
- net GND: now also J6.2 (Pin_2)
- net LIDAR_M_CTR: now also J6.1 (Pin_1)
- net LIDAR_TX: now also J6.4 (Pin_4)
- no-connect marks 3 -> 4
Changed lines of the file:
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@@
 	)
 	(no_connect
+		(at 187.96 55.88)
+	)
+	(no_connect
 		(at 100.33 110.49)
 	)
@@
 	(wire
 		(pts
+			(xy 187.96 60.96) (xy 196.85 60.96)
+		)
+		(stroke
+			(width 0)
+			(type default)
+		)
+	)
+	(wire
+		(pts
 			(xy 36.83 106.68) (xy 46.99 106.68)
 		)
@@
 	(wire
 		(pts
-			(xy 187.96 58.42) (xy 196.85 58.42)
-		)
-		(stroke
-			(width 0)
-			(type default)
-		)
-	)
-	(wire
-		(pts
 			(xy 224.79 109.22) (xy 224.79 111.76)
 		)
@@
 	(wire
 		(pts
-			(xy 187.96 55.88) (xy 196.85 55.88)
+			(xy 195.58 111.76) (xy 198.12 111.76)
 		)
 		(stroke
@@
 	(wire
 		(pts
-			(xy 195.58 111.76) (xy 198.12 111.76)
+			(xy 226.06 140.97) (xy 231.14 140.97)
 		)
 		(stroke
@@
 	(wire
 		(pts
-			(xy 226.06 140.97) (xy 231.14 140.97)
+			(xy 46.99 106.68) (xy 60.96 106.68)
 		)
 		(stroke
@@
 	(wire
 		(pts
-			(xy 46.99 106.68) (xy 60.96 106.68)
+			(xy 184.15 111.76) (xy 189.23 111.76)
 		)
 		(stroke
@@
 	(wire
 		(pts
-			(xy 184.15 111.76) (xy 189.23 111.76)
+			(xy 100.33 85.09) (xy 100.33 78.74)
 		)
 		(stroke
@@
 	(wire
 		(pts
-			(xy 100.33 85.09) (xy 100.33 78.74)
+			(xy 195.58 119.38) (xy 186.69 119.38)
 		)
 		(stroke
@@
 	(wire
 		(pts
-			(xy 195.58 119.38) (xy 186.69 119.38)
+			(xy 187.96 58.42) (xy 196.85 58.42)
 		)
 		(stroke
@@
 	(hierarchical_label "LIDAR_M_CTR"
 		(shape input)
-		(at 196.85 58.42 0)
+		(at 196.85 60.96 0)
 		(effects
 			(font
@@
 			)
 		)
-		(property "Footprint" "Capacitor_SMD:C_01005_0402Metric"
+		(property "Footprint" "Capacitor_SMD:C_0402_1005Metric"
 			(at 237.1852 119.38 0)
 			(effects
@@
 			)
 		)
-		(property "Footprint" "Capacitor_SMD:C_01005_0402Metric"
+		(property "Footprint" "Capacitor_SMD:C_0402_1005Metric"
 			(at 88.9 73.66 0)
 			(effects
@@
 			)
 		)
-		(property "Footprint" "Capacitor_SMD:C_01005_0402Metric"
+		(property "Footprint" "Capacitor_SMD:C_0402_1005Metric"
 			(at 196.5452 119.38 0)
 			(effects
@@
 			)
 		)
-		(property "Footprint" "Capacitor_SMD:C_01005_0402Metric"
+		(property "Footprint" "Capacitor_SMD:C_0402_1005Metric"
 			(at 107.95 76.2 0)
 			(effects
@@
 			)
 		)
-		(property "Footprint" "Capacitor_SMD:C_01005_0402Metric"
+		(property "Footprint" "Capacitor_SMD:C_0402_1005Metric"
 			(at 238.4552 148.59 0)
 			(effects
@@
 	)
 	(symbol
-		(lib_id "Connector_Generic:Conn_01x04")
-		(at 182.88 55.88 180)
+		(lib_id "Sensor_Motion:ADXL343")
+		(at 95.25 97.79 0)
 		(unit 1)
 		(exclude_from_sim no)
@@
 		(dnp no)
 		(fields_autoplaced yes)
-		(property "Reference" "J10"
-			(at 182.88 44.45 0)
+		(property "Reference" "U4"
+			(at 110.49 91.3698 0)
 			(effects
 				(font
@@
 			)
 		)
-		(property "Value" "Conn_01x04"
-			(at 182.88 46.99 0)
+		(property "Value" "ADXL343"
+			(at 110.49 93.9098 0)
 			(effects
 				(font
@@
 			)
 		)
-		(property "Footprint" "Connector_JST:JST_XH_S4B-XH-A_1x04_P2.50mm_Horizontal"
-			(at 182.88 55.88 0)
+		(property "Footprint" "Package_LGA:LGA-14_3x5mm_P0.8mm_LayoutBorder1x6y"
+			(at 95.25 97.79 0)
 			(effects
 				(font
@@
 			)
 		)
-		(property "Datasheet" "~"
-			(at 182.88 55.88 0)
+		(property "Datasheet" "https://www.analog.com/media/en/technical-documentation/data-sheets/ADXL343.pdf"
+			(at 95.25 97.79 0)
 			(effects
 				(font
@@
 			)
 		)
-		(property "Description" "Generic connector, single row, 01x04, script generated (kicad-library-utils/schlib/autogen/connector/)"
-			(at 182.88 55.88 0)
+		(property "Description" "3-Axis MEMS Accelerometer, 2/4/8/16g range, I2C/SPI, LGA-14"
+			(at 95.25 97.79 0)
 			(effects
 				(font
@@
 			)
 		)
+		(pin "3"
+		)
+		(pin "14"
+		)
+		(pin "13"
+		)
+		(pin "7"
+		)
+		(pin "12"
+		)
 		(pin "1"
 		)
-		(pin "4"
+		(pin "8"
 		)
-		(pin "3"
+		(pin "11"
+		)
+		(pin "6"
+		)
+		(pin "9"
 		)
 		(pin "2"
 		)
+		(pin "5"
+		)
+		(pin "10"
+		)
+		(pin "4"
+		)
 		(instances
-			(project ""
+			(project "projet"
 				(path "/b2330267-3262-4d12-877e-36612b3f2d84/fb3a1801-63de-4558-9fb3-e6b98a5f4817"
-					(reference "J10")
+					(reference "U4")
 					(unit 1)
 				)
@@
 	)
 	(symbol
-		(lib_id "Sensor_Motion:ADXL343")
-		(at 95.25 97.79 0)
+		(lib_id "Connector_Generic:Conn_01x05")
+		(at 182.88 55.88 180)
 		(unit 1)
 		(exclude_from_sim no)
@@
 		(dnp no)
 		(fields_autoplaced yes)
-		(property "Reference" "U4"
-			(at 110.49 91.3698 0)
+		(property "Reference" "J6"
+			(at 182.88 44.45 0)
 			(effects
 				(font
@@
 			)
 		)
-		(property "Value" "ADXL343"
-			(at 110.49 93.9098 0)
+		(property "Value" "Conn_01x05"
+			(at 182.88 46.99 0)
 			(effects
 				(font
@@
 			)
 		)
-		(property "Footprint" "Package_LGA:LGA-14_3x5mm_P0.8mm_LayoutBorder1x6y"
-			(at 95.25 97.79 0)
+		(property "Footprint" ""
+			(at 182.88 55.88 0)
 			(effects
 				(font
@@
 			)
 		)
-		(property "Datasheet" "https://www.analog.com/media/en/technical-documentation/data-sheets/ADXL343.pdf"
-			(at 95.25 97.79 0)
+		(property "Datasheet" "~"
+			(at 182.88 55.88 0)
 			(effects
 				(font
@@
 			)
 		)
-		(property "Description" "3-Axis MEMS Accelerometer, 2/4/8/16g range, I2C/SPI, LGA-14"
-			(at 95.25 97.79 0)
+		(property "Description" "Generic connector, single row, 01x05, script generated (kicad-library-utils/schlib/autogen/connector/)"
+			(at 182.88 55.88 0)
 			(effects
 				(font
@@
 			)
 		)
-		(pin "3"
-		)
-		(pin "14"
-		)
-		(pin "13"
-		)
-		(pin "7"
-		)
-		(pin "12"
-		)
-		(pin "1"
-		)
-		(pin "8"
-		)
-		(pin "11"
-		)
-		(pin "6"
+		(pin "5"
 		)
-		(pin "9"
+		(pin "4"
 		)
 		(pin "2"
 		)
-		(pin "5"
-		)
-		(pin "10"
+		(pin "1"
 		)
-		(pin "4"
+		(pin "3"
 		)
 		(instances
 			(project "projet"
 				(path "/b2330267-3262-4d12-877e-36612b3f2d84/fb3a1801-63de-4558-9fb3-e6b98a5f4817"
-					(reference "U4")
+					(reference "J6")
 					(unit 1)
 				)
@@
 			)
 		)
-		(property "Footprint" "Capacitor_SMD:C_01005_0402Metric"
+		(property "Footprint" "Capacitor_SMD:C_0402_1005Metric"
 			(at 195.2752 149.86 0)
 			(effects
@@
 	(symbol
 		(lib_id "power:GND")
-		(at 196.85 55.88 90)
+		(at 196.85 58.42 90)
 		(unit 1)
 		(exclude_from_sim no)
@@
 		(fields_autoplaced yes)
 		(property "Reference" "#PWR047"
-			(at 203.2 55.88 0)
+			(at 203.2 58.42 0)
 			(effects
 				(font
@@
 		)
 		(property "Value" "GND"
-			(at 200.66 55.8799 90)
+			(at 200.66 58.4199 90)
 			(effects
 				(font
@@
 		)
 		(property "Footprint" ""
-			(at 196.85 55.88 0)
+			(at 196.85 58.42 0)
 			(effects
 				(font
@@
 		)
 		(property "Datasheet" ""
-			(at 196.85 55.88 0)
+			(at 196.85 58.42 0)
 			(effects
 				(font
@@
 		)
 		(property "Description" "Power symbol creates a global label with name \"GND\" , ground"
-			(at 196.85 55.88 0)
+			(at 196.85 58.42 0)
 			(effects
 				(font
