File: Projet_Robot_Autonome/ProjetX.kicad_sch (KiCad schematic)
At the start: 4 parts

Commit message: Updated KiCad project files
Other:
- sheet STM32 ports: added none; removed BORDER_5, BORDER_6
- sheet Sensors ports: added none; removed BORDER_5, BORDER_6
Changed lines of the file:
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@@
-	(wire
-		(pts
-			(xy 100.33 87.63) (xy 123.19 87.63)
-		)
-		(stroke
-			(width 0)
-			(type default)
-		)
-	)
 	(wire
 		(pts
@@
 		(pts
 			(xy 100.33 74.93) (xy 123.19 74.93)
-		)
-		(stroke
-			(width 0)
-			(type default)
-		)
-	)
-	(wire
-		(pts
-			(xy 100.33 90.17) (xy 123.19 90.17)
 		)
 		(stroke
@@
 			)
 		)
-		(pin "BORDER_5" input
-			(at 123.19 87.63 180)
-			(effects
-				(font
-					(size 1.27 1.27)
-				)
-				(justify left)
-			)
-		)
-		(pin "BORDER_6" input
-			(at 123.19 90.17 180)
-			(effects
-				(font
-					(size 1.27 1.27)
-				)
-				(justify left)
-			)
-		)
 		(instances
 			(project "ProjetX"
@@
 			(effects
 				(font
-					(size 1.27 1.27)
-				)
-				(justify right)
-			)
-		)
-		(pin "BORDER_5" output
-			(at 100.33 87.63 0)
-			(effects
-				(font
-					(size 1.27 1.27)
-				)
-				(justify right)
-			)
-		)
-		(pin "BORDER_6" output
-			(at 100.33 90.17 0)
-			(effects
-				(font
