File: Projet_Robot_Autonome/Sensors.kicad_sch (KiCad schematic)
At the start: 25 parts, among them J11 Conn_01x05, J4 BORDER, J6 Conn_01x05, J7 BORDER, J8 BORDER, J9 BORDER, U4 ADXL343

Commit message: Updated KiCad project files
Parts:
- added R26: 470R, Resistor_SMD:R_0402_1005Metric, symbol Device:R_Small
Connections:
- net LIDAR_TX: now also R26.2; no longer J6.4 (Pin_4)
- new net: J6.4 (Pin_4), R26.1
Changed lines of the file:
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@@
+	(wire
+		(pts
+			(xy 201.93 53.34) (xy 208.28 53.34)
+		)
+		(stroke
+			(width 0)
+			(type default)
+		)
+	)
 	(wire
 		(pts
@@
 	(hierarchical_label "LIDAR_TX"
 		(shape output)
-		(at 196.85 53.34 0)
+		(at 208.28 53.34 0)
 		(effects
 			(font
@@
 					(unit 1)
 				)
+			)
+		)
+	)
+	(symbol
+		(lib_id "Device:R_Small")
+		(at 199.39 53.34 90)
+		(mirror x)
+		(unit 1)
+		(exclude_from_sim no)
+		(in_bom yes)
+		(on_board yes)
+		(dnp no)
+		(property "Reference" "R26"
+			(at 199.39 58.42 90)
+			(effects
+				(font
+					(size 1.016 1.016)
+				)
+			)
+		)
+		(property "Value" "470R"
+			(at 199.39 55.88 90)
+			(effects
+				(font
+					(size 1.27 1.27)
+				)
+			)
+		)
+		(property "Footprint" "Resistor_SMD:R_0402_1005Metric"
+			(at 199.39 53.34 0)
+			(effects
+				(font
+					(size 1.27 1.27)
+				)
+				(hide yes)
+			)
+		)
+		(property "Datasheet" "~"
+			(at 199.39 53.34 0)
+			(effects
+				(font
+					(size 1.27 1.27)
+				)
+				(hide yes)
+			)
+		)
+		(property "Description" "Resistor, small symbol"
+			(at 199.39 53.34 0)
+			(effects
+				(font
+					(size 1.27 1.27)
+				)
+				(hide yes)
+			)
+		)
+		(pin "1"
+		)
+		(pin "2"
+		)
+		(instances
+			(project ""
+				(path "/b2330267-3262-4d12-877e-36612b3f2d84/fb3a1801-63de-4558-9fb3-e6b98a5f4817"
+					(reference "R26")
+					(unit 1)
+				)
