File: Projet_Robot_Autonome/Alimentation.kicad_sch (KiCad schematic)
At the start: 28 parts, among them IC1 MP1475DJ-LF-P, J2 Screw_Terminal_01x02, SW1 ON/OFF

Commit message: Updated KiCad project files
Parts:
- removed C28, C29: 22uF, Capacitor_SMD:C_0402_1005Metric, symbol Device:C_Small
- added C36, C37: 22uF, Capacitor_SMD:C_0805_2012Metric, symbol Device:C_Small
- C24: footprint Capacitor_SMD:C_0402_1005Metric -> Capacitor_SMD:C_0805_2012Metric
Connections:
- net +5V: now also C36.1, C37.1
- net GND: now also C36.2, C37.2
Changed lines of the file:
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@@
 	)
 	(junction
-		(at 195.58 63.5)
+		(at 195.58 68.58)
 		(diameter 0)
 		(color 0 0 0 0)
 	)
 	(junction
-		(at 162.56 63.5)
+		(at 195.58 63.5)
 		(diameter 0)
 		(color 0 0 0 0)
 	)
 	(junction
-		(at 218.44 57.15)
+		(at 162.56 63.5)
 		(diameter 0)
 		(color 0 0 0 0)
 	)
 	(junction
-		(at 33.02 82.55)
+		(at 218.44 57.15)
 		(diameter 0)
 		(color 0 0 0 0)
 	)
 	(junction
-		(at 195.58 68.58)
+		(at 33.02 82.55)
 		(diameter 0)
 		(color 0 0 0 0)
@@
 	)
 	(junction
-		(at 184.15 63.5)
+		(at 91.44 58.42)
 		(diameter 0)
 		(color 0 0 0 0)
 	)
 	(junction
-		(at 91.44 58.42)
+		(at 184.15 63.5)
 		(diameter 0)
 		(color 0 0 0 0)
@@
 	(wire
 		(pts
-			(xy 184.15 63.5) (xy 195.58 63.5)
+			(xy 45.72 93.98) (xy 50.8 93.98)
 		)
 		(stroke
@@
 	(wire
 		(pts
-			(xy 45.72 93.98) (xy 50.8 93.98)
+			(xy 218.44 57.15) (xy 227.33 57.15)
 		)
 		(stroke
@@
 	(wire
 		(pts
-			(xy 218.44 57.15) (xy 227.33 57.15)
+			(xy 45.72 82.55) (xy 50.8 82.55)
 		)
 		(stroke
@@
 	(wire
 		(pts
-			(xy 45.72 82.55) (xy 50.8 82.55)
+			(xy 82.55 63.5) (xy 91.44 63.5)
 		)
 		(stroke
@@
 	(wire
 		(pts
-			(xy 82.55 63.5) (xy 91.44 63.5)
+			(xy 162.56 63.5) (xy 170.18 63.5)
 		)
 		(stroke
@@
 	(wire
 		(pts
-			(xy 162.56 63.5) (xy 170.18 63.5)
+			(xy 184.15 63.5) (xy 195.58 63.5)
 		)
 		(stroke
@@
 	(symbol
 		(lib_id "Device:C_Small")
+		(at 184.15 66.04 0)
+		(unit 1)
+		(exclude_from_sim no)
+		(in_bom yes)
+		(on_board yes)
+		(dnp no)
+		(fields_autoplaced yes)
+		(property "Reference" "C37"
+			(at 186.69 64.7762 0)
+			(effects
+				(font
+					(size 1.27 1.27)
+				)
+				(justify left)
+			)
+		)
+		(property "Value" "22uF"
+			(at 186.69 67.3162 0)
+			(effects
+				(font
+					(size 1.27 1.27)
+				)
+				(justify left)
+			)
+		)
+		(property "Footprint" "Capacitor_SMD:C_0805_2012Metric"
+			(at 184.15 66.04 0)
+			(effects
+				(font
+					(size 1.27 1.27)
+				)
+				(hide yes)
+			)
+		)
+		(property "Datasheet" "~"
+			(at 184.15 66.04 0)
+			(effects
+				(font
+					(size 1.27 1.27)
+				)
+				(hide yes)
+			)
+		)
+		(property "Description" "Unpolarized capacitor, small symbol"
+			(at 184.15 66.04 0)
+			(effects
+				(font
+					(size 1.27 1.27)
+				)
+				(hide yes)
+			)
+		)
+		(pin "1"
+		)
+		(pin "2"
+		)
+		(instances
+			(project "ProjetX"
+				(path "/b2330267-3262-4d12-877e-36612b3f2d84/027c0f16-9d10-4b80-857c-f21dafef43b8"
+					(reference "C37")
+					(unit 1)
+				)
+			)
+		)
+	)
+	(symbol
+		(lib_id "Device:C_Small")
 		(at 91.44 60.96 0)
 		(unit 1)
@@
 			)
 		)
-		(property "Footprint" "Capacitor_SMD:C_0402_1005Metric"
+		(property "Footprint" "Capacitor_SMD:C_0805_2012Metric"
 			(at 82.55 60.96 0)
 			(effects
@@
 	)
 	(symbol
+		(lib_id "Device:C_Small")
+		(at 195.58 66.04 0)
+		(unit 1)
+		(exclude_from_sim no)
+		(in_bom yes)
+		(on_board yes)
+		(dnp no)
+		(fields_autoplaced yes)
+		(property "Reference" "C36"
+			(at 198.12 64.7762 0)
+			(effects
+				(font
+					(size 1.27 1.27)
+				)
+				(justify left)
+			)
+		)
+		(property "Value" "22uF"
+			(at 198.12 67.3162 0)
+			(effects
+				(font
+					(size 1.27 1.27)
+				)
+				(justify left)
+			)
+		)
+		(property "Footprint" "Capacitor_SMD:C_0805_2012Metric"
+			(at 195.58 66.04 0)
+			(effects
+				(font
+					(size 1.27 1.27)
+				)
+				(hide yes)
+			)
+		)
+		(property "Datasheet" "~"
+			(at 195.58 66.04 0)
+			(effects
+				(font
+					(size 1.27 1.27)
+				)
+				(hide yes)
+			)
+		)
+		(property "Description" "Unpolarized capacitor, small symbol"
+			(at 195.58 66.04 0)
+			(effects
+				(font
+					(size 1.27 1.27)
+				)
+				(hide yes)
+			)
+		)
+		(pin "1"
+		)
+		(pin "2"
+		)
+		(instances
+			(project "ProjetX"
+				(path "/b2330267-3262-4d12-877e-36612b3f2d84/027c0f16-9d10-4b80-857c-f21dafef43b8"
+					(reference "C36")
+					(unit 1)
+				)
+			)
+		)
+	)
+	(symbol
 		(lib_id "power:GND")
 		(at 218.44 71.12 0)
@@
 	)
 	(symbol
-		(lib_id "Device:C_Small")
-		(at 184.15 66.04 0)
-		(unit 1)
-		(exclude_from_sim no)
-		(in_bom yes)
-		(on_board yes)
-		(dnp no)
-		(fields_autoplaced yes)
-		(property "Reference" "C28"
-			(at 186.69 64.7762 0)
-			(effects
-				(font
-					(size 1.27 1.27)
-				)
-				(justify left)
-			)
-		)
-		(property "Value" "22uF"
-			(at 186.69 67.3162 0)
-			(effects
-				(font
-					(size 1.27 1.27)
-				)
-				(justify left)
-			)
-		)
-		(property "Footprint" "Capacitor_SMD:C_0402_1005Metric"
-			(at 184.15 66.04 0)
-			(effects
-				(font
-					(size 1.27 1.27)
-				)
-				(hide yes)
-			)
-		)
-		(property "Datasheet" "~"
-			(at 184.15 66.04 0)
-			(effects
-				(font
-					(size 1.27 1.27)
-				)
-				(hide yes)
-			)
-		)
-		(property "Description" "Unpolarized capacitor, small symbol"
-			(at 184.15 66.04 0)
-			(effects
-				(font
-					(size 1.27 1.27)
-				)
-				(hide yes)
-			)
-		)
-		(pin "1"
-		)
-		(pin "2"
-		)
-		(instances
-			(project "projet"
-				(path "/b2330267-3262-4d12-877e-36612b3f2d84/027c0f16-9d10-4b80-857c-f21dafef43b8"
-					(reference "C28")
-					(unit 1)
-				)
-			)
-		)
-	)
-	(symbol
 		(lib_id "power:+BATT")
 		(at 69.85 45.72 0)
@@
 					(unit 1)
 				)
-			)
-		)
-	)
-	(symbol
-		(lib_id "Device:C_Small")
-		(at 195.58 66.04 0)
-		(unit 1)
-		(exclude_from_sim no)
-		(in_bom yes)
-		(on_board yes)
-		(dnp no)
-		(fields_autoplaced yes)
-		(property "Reference" "C29"
-			(at 198.12 64.7762 0)
-			(effects
-				(font
-					(size 1.27 1.27)
-				)
-				(justify left)
-			)
-		)
-		(property "Value" "22uF"
-			(at 198.12 67.3162 0)
-			(effects
-				(font
-					(size 1.27 1.27)
-				)
-				(justify left)
-			)
-		)
-		(property "Footprint" "Capacitor_SMD:C_0402_1005Metric"
-			(at 195.58 66.04 0)
-			(effects
-				(font
-					(size 1.27 1.27)
-				)
-				(hide yes)
-			)
-		)
-		(property "Datasheet" "~"
-			(at 195.58 66.04 0)
-			(effects
-				(font
-					(size 1.27 1.27)
-				)
-				(hide yes)
-			)
-		)
-		(property "Description" "Unpolarized capacitor, small symbol"
-			(at 195.58 66.04 0)
-			(effects
-				(font
-					(size 1.27 1.27)
-				)
-				(hide yes)
-			)
-		)
-		(pin "1"
-		)
-		(pin "2"
-		)
-		(instances
-			(project "projet"
-				(path "/b2330267-3262-4d12-877e-36612b3f2d84/027c0f16-9d10-4b80-857c-f21dafef43b8"
-					(reference "C29")
-					(unit 1)
-				)

Commit message: Updated KiCad project files
Parts:
- removed SW1: ON/OFF, Button_Switch_SMD:Nidec_Copal_CAS-120A, symbol Switch:SW_Nidec_CAS-120A1
- added S1: 1101M2S3CQE2, swithes:sw wurth, symbol 1101M2S3CQE2:1101M2S3CQE2
Connections:
- net +BATT: now also S1.2
- net GND: now also J2.1 (Pin_1); no longer J2.2 (Pin_2)
- new net: J2.2 (Pin_2), S1.3
Other:
- moved on the sheet: D1_PWR_BATT1, D2_PWR_5V1, D3_PWR_3V1, J2, R2, R3, R4
