File: Projet_Robot_Autonome/ProjetX.kicad_pcb (KiCad board)
At the start: 4 copper layers, 96 parts, among them IC1 MP1475DJ-LF-P, J1 Conn_ST_STDC14, J11 Conn_01x05, J2 Screw_Terminal_01x02, J3 Conn_01x06, J4 BORDER, J5 Conn_01x06, J6 Conn_01x05, J7 BORDER, J8 BORDER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

Commit message: Updated KiCad project files
Parts:
- removed C28, C29: 22uF, Capacitor_SMD:C_0402_1005Metric
- removed JP1, JP2: SolderJumper_2_Open, Jumper:SolderJumper-2_P1.3mm_Open_RoundedPad1.0x1.5mm
- added C35: 100n, Capacitor_SMD:C_0402_1005Metric, F.Cu at (144.1, 100.2)
- added C36: 22uF, Capacitor_SMD:C_0805_2012Metric, F.Cu at (167.5, 106.8)
- added C37: 22uF, Capacitor_SMD:C_0805_2012Metric, F.Cu at (169.7, 106.8)
- added R24: 1k, Resistor_SMD:R_0402_1005Metric, F.Cu at (144.1, 101.3)
- added R25: 1k, Resistor_SMD:R_0402_1005Metric, F.Cu at (143.7, 102.9)
- added R26: 470R, Resistor_SMD:R_0402_1005Metric, F.Cu at (150.8, 89.0)
- added SW2: SW_Push, Button_Switch_THT:SW_PUSH_6mm_H9.5mm, F.Cu at (136.7, 104.5)
- C14, C18: footprint Capacitor_SMD:C_0402_1005Metric -> Capacitor_SMD:C_0603_1608Metric
- C24: footprint Capacitor_SMD:C_0402_1005Metric -> Capacitor_SMD:C_0805_2012Metric
- moved SW1 54.7 mm to (181.4, 122.3)
- moved J11 41.7 mm to (174.2, 85.1), turned to 180 degrees
- moved J2 38.3 mm to (171.1, 119.1), turned to 0 degrees
- moved J7 36.8 mm to (153.7, 119.1), turned to 0 degrees
- moved J8 36.8 mm to (145.2, 119.1), turned to 0 degrees
- moved J9 36.1 mm to (162.2, 119.1), turned to 0 degrees
- moved J6 34.7 mm to (158.2, 85.1), turned to 180 degrees
- moved R11 31.8 mm to (168.9, 114.2)
- moved J4 31.7 mm to (144.9, 91.0), turned to -90 degrees
- moved R17 30.0 mm to (155.0, 115.7), turned to 0 degrees
- moved R12 30.0 mm to (164.3, 109.8), turned to 180 degrees
- moved R16 29.4 mm to (153.0, 115.7)
- moved R21 28.9 mm to (149.0, 115.7), turned to 0 degrees
- moved R20 28.8 mm to (147.0, 115.7)
- moved C34 28.5 mm to (161.8, 115.7), turned to 0 degrees
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Connections:
- J1 pad 13: Net-(J1-VCP_RX) -> /STM32/RX_SWD
- J1 pad 14: Net-(J1-VCP_TX) -> /STM32/TX_SWD
- J6 pad 4: /STM32/LIDAR_TX -> Net-(J6-Pin_4)
- U1 pad 10: /STM32/BORDER_3 -> unconnected-(U1-PA2-Pad10)
- U1 pad 13: unconnected-(U1-PA5-Pad13) -> /STM32/BORDER_3
- U1 pad 14: /STM32/INT1_ACC -> /STM32/INT2_ACC
- U1 pad 15: /STM32/INT2_ACC -> /STM32/INT1_ACC
- U1 pad 26: /STM32/SCL -> /Actionneurs/REV2
- U1 pad 27: /STM32/SDA -> /Actionneurs/REV1
- U1 pad 29: unconnected-(U1-PC6-Pad29) -> /Actionneurs/ENCOD_B2
- U1 pad 30: /Actionneurs/FWD1 -> /Actionneurs/FWD2
- U1 pad 31: /Actionneurs/FWD2 -> /Actionneurs/FWD1
- U1 pad 33: unconnected-(U1-PA11-Pad33) -> /Actionneurs/ENCOD_B1
- U1 pad 34: unconnected-(U1-PA12-Pad34) -> /Actionneurs/ENCOD_A1
- U1 pad 38: unconnected-(U1-PA15-Pad38) -> /STM32/CHAT/SOURIS
- U1 pad 42: /Actionneurs/ENCOD_B1 -> unconnected-(U1-PB4-Pad42)
- U1 pad 43: /Actionneurs/ENCOD_A1 -> /Actionneurs/ENCOD_A2
- U1 pad 44: /Actionneurs/ENCOD_A2 -> unconnected-(U1-PB6-Pad44)
- U1 pad 45: /Actionneurs/ENCOD_B2 -> unconnected-(U1-PB7-Pad45)
- U1 pad 46: /Actionneurs/REV1 -> /STM32/SCL
- U1 pad 47: /Actionneurs/REV2 -> /STM32/SDA
Routing:
- net /Actionneurs/ENCOD_B2: track 0.00 -> 72.1 mm, vias 0 -> 2
- net /Actionneurs/FWD2: track 0.00 -> 64.0 mm
- net GND: track 0.00 -> 62.0 mm, vias 0 -> 29
- net /Actionneurs/ENCOD_A2: track 0.00 -> 60.5 mm
- net /Actionneurs/FWD1: track 0.00 -> 49.8 mm
- net +3.3V: track 0.00 -> 39.8 mm, vias 0 -> 14
- net /Actionneurs/ENCOD_B1: track 0.00 -> 37.4 mm, vias 0 -> 2
- net /Actionneurs/ENCOD_A1: track 0.00 -> 36.8 mm, vias 0 -> 2
- net /STM32/SCL: track 0.00 -> 35.4 mm
- net /STM32/SDA: track 0.00 -> 30.5 mm
- net /Actionneurs/REV1: track 0.00 -> 28.3 mm, vias 0 -> 4
- net /STM32/BLE_RX: track 0.00 -> 28.1 mm, vias 0 -> 2
- net /Actionneurs/REV2: track 0.00 -> 27.6 mm, vias 0 -> 2
- net /STM32/LIDAR_TX: track 0.00 -> 27.1 mm, vias 0 -> 2
- net /STM32/BORDER_4: track 0.00 -> 25.3 mm, vias 0 -> 2
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- added copper zone on In2.Cu, net +3.3V
- added copper zone on In2.Cu, net +5V
- added copper zone on In2.Cu, net +BATT
- added copper zone on B.Cu, net GND
- added copper zone on F.Cu, net GND

Commit message: Updated KiCad project files
Routing:
- net Net-(J2-Pin_1): track 11.3 -> 13.1 mm
- net /Actionneurs/ENCOD_B2: track 72.1 -> 73.2 mm
- net GND: track 62.0 -> 62.4 mm, vias 29 -> 38

Commit message: Updated KiCad project files
Other:
- board outline added: 57 x 54 mm
Changed lines of the file:
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@@
 		(stroke
 			(width 0.1)
-			(type default)
+			(type solid)
 		)
-		(layer "F.SilkS")
+		(layer "Edge.Cuts")
 	)
 	(gr_arc
@@
 		(stroke
 			(width 0.1)
-			(type default)
+			(type solid)
 		)
-		(layer "F.SilkS")
+		(layer "Edge.Cuts")
 	)
 	(gr_line
@@
 		(stroke
 			(width 0.1)
-			(type default)
+			(type solid)
 		)
-		(layer "F.SilkS")
+		(layer "Edge.Cuts")
 	)
 	(gr_arc
@@
 		(stroke
 			(width 0.1)
-			(type default)
+			(type solid)
 		)
-		(layer "F.SilkS")
+		(layer "Edge.Cuts")
 	)
 	(gr_line
@@
 		(stroke
 			(width 0.1)
-			(type default)
+			(type solid)
 		)
-		(layer "F.SilkS")
+		(layer "Edge.Cuts")
 	)
 	(gr_line
@@
 		(stroke
 			(width 0.1)
-			(type default)
+			(type solid)
 		)
-		(layer "F.SilkS")
+		(layer "Edge.Cuts")
 	)
 	(gr_arc
@@
 		(stroke
 			(width 0.1)
-			(type default)
+			(type solid)
 		)
-		(layer "F.SilkS")
+		(layer "Edge.Cuts")
 	)
 	(gr_line
@@
 		(stroke
 			(width 0.1)
-			(type default)
+			(type solid)
 		)
-		(layer "F.SilkS")
+		(layer "Edge.Cuts")
 	)
 	(segment
@@
 		(polygon
 			(pts
-				(xy 135.1 75.1) (xy 192 75.1) (xy 192 128.9) (xy 135.1 128.9)
+				(xy 134 74.1) (xy 192 74.8) (xy 192.5 129.3) (xy 134.1 129.6)
 			)
 		)
@@
 		(polygon
 			(pts
-				(xy 135.093956 75.181184) (xy 135.4 128.9) (xy 192 128.8) (xy 191.79138 75)
+				(xy 134.3 74.4) (xy 134.6 129.2) (xy 192.8 129.5) (xy 192.2 74.6)
 			)
 		)
@@
 		(polygon
 			(pts
-				(xy 135.493801 75.20105) (xy 191.9 75.1) (xy 191.812361 128.863805) (xy 135.1 128.9)
+				(xy 134.6 74.6) (xy 192.1 74.7) (xy 193.1 129.8) (xy 134.4 129.4)
 			)
 		)

Commit message: Updated KiCad project files
Parts:
- removed SW1: ON/OFF, Button_Switch_SMD:Nidec_Copal_CAS-120A
- added S1: 1101M2S3CQE2, swithes:sw wurth, F.Cu at (179.8, 121.6)
- SW2: footprint Button_Switch_THT:SW_PUSH_6mm_H9.5mm -> Button_Switch_SMD:SW_Push_1P1T_NO_E-Switch_TL3301NxxxxxG
- moved H3 49.6 mm to (139.0, 125.0)
- moved H4 49.5 mm to (188.0, 125.0)
- moved R3 24.3 mm to (175.5, 103.6)
- moved D2_PWR_5V1 24.3 mm to (175.5, 100.9)
- moved D1_PWR_BATT1 24.3 mm to (177.6, 101.0)
- moved D3_PWR_3V1 24.3 mm to (173.3, 100.9)
- moved R2 24.3 mm to (177.6, 103.7)
- moved R4 24.3 mm to (173.3, 103.6)
- moved R15 22.8 mm to (170.0, 93.1), turned to 0 degrees
- moved C30 22.1 mm to (167.9, 92.1), turned to 180 degrees
- moved R13 21.3 mm to (167.9, 93.2), turned to 180 degrees
- moved R11 20.9 mm to (174.4, 94.0)
- moved R10 20.7 mm to (170.0, 91.0)
- moved R12 20.7 mm to (170.0, 90.0)
- moved C26 20.7 mm to (170.0, 92.1)
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Connections:
- J2 pad 1: Net-(J2-Pin_1) -> GND
- J2 pad 2: GND -> Net-(J2-Pin_2)
Routing:
- net /Actionneurs/ENCOD_B2: track 73.2 -> 44.9 mm, vias 2 -> 1
- net +3.3V: track 39.8 -> 67.7 mm, vias 14 -> 18
- net /Actionneurs/FWD2: track 64.0 -> 41.0 mm, vias 0 -> 2
- net +BATT: track 21.0 -> 42.1 mm, vias 9 -> 11
- net /Actionneurs/REV2: track 27.6 -> 43.8 mm
- net /Actionneurs/FWD1: track 49.8 -> 35.8 mm, vias 0 -> 2
- net Net-(J2-Pin_1): track 13.1 -> 0.00 mm
- net Net-(J2-Pin_2): track 0.00 -> 11.6 mm
- net GND: track 62.4 -> 72.7 mm, vias 38 -> 36
- net +5V: track 15.8 -> 23.6 mm, vias 6 -> 3
- net /STM32/LIDAR_TX: track 27.1 -> 33.4 mm
- net /STM32/BLE_RX: track 28.1 -> 33.5 mm, vias 2 -> 0
- net /Actionneurs/ENCOD_A1: track 36.8 -> 42.0 mm, vias 2 -> 1
- net /Actionneurs/ENCOD_B1: track 37.4 -> 42.4 mm, vias 2 -> 1
- net /STM32/BORDER_4: track 25.3 -> 20.4 mm
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