File: Projet_Robot_Autonome/STM32.kicad_sch (KiCad schematic)
At the start: 23 parts, among them J1 Conn_ST_STDC14, U1 STM32G431CBUx, Y1 Crystal_GND24_Small

Commit message: Updated KiCad project files
Parts:
- removed JP1, JP2: SolderJumper_2_Open, Jumper:SolderJumper-2_P1.3mm_Open_RoundedPad1.0x1.5mm, symbol Jumper:SolderJumper_2_Open
- added C35: 100n, Capacitor_SMD:C_0402_1005Metric, symbol Device:C_Small
- added R24, R25: 1k, Resistor_SMD:R_0402_1005Metric, symbol Device:R_Small
- added SW2: SW_Push, Button_Switch_THT:SW_PUSH_6mm_H9.5mm, symbol Switch:SW_Push
Connections:
- net +3.3V: now also R25.2
- net BORDER_3: now also U1.13 (PA5); no longer U1.10 (PA2)
- net ENCOD_A1: now also U1.34 (PA12); no longer U1.43 (PB5)
- net ENCOD_A2: now also U1.43 (PB5); no longer U1.44 (PB6)
- net ENCOD_B1: now also U1.33 (PA11); no longer U1.42 (PB4)
- net ENCOD_B2: now also U1.29 (PC6); no longer U1.45 (PB7)
- net FWD1: now also U1.31 (PA9); no longer U1.30 (PA8)
- net FWD2: now also U1.30 (PA8); no longer U1.31 (PA9)
- net GND: now also C35.2, SW2.2
- net INT1_ACC: now also U1.15 (PA7); no longer U1.14 (PA6)
- net INT2_ACC: now also U1.14 (PA6); no longer U1.15 (PA7)
- net REV1: now also U1.27 (PB14); no longer U1.46 (PB8)
- net REV2: now also U1.26 (PB13); no longer U1.47 (PB9)
- net RX_SWD: now also J1.13 (VCP_RX)
- net SCL: now also U1.46 (PB8); no longer U1.26 (PB13)
- net SDA: now also U1.47 (PB9); no longer U1.27 (PB14)
- net TX_SWD: now also J1.14 (VCP_TX)
- net CHAT/SOURIS: now reaches U1.38 (PA15)
- net CHAT/SOURIS: now also C35.1, R24.1
- new net: R24.2, R25.1, SW2.1
- no-connect marks 13 -> 12

Commit message: Updated KiCad project files
Parts:
- SW2: footprint Button_Switch_THT:SW_PUSH_6mm_H9.5mm -> Button_Switch_SMD:SW_Push_1P1T_NO_E-Switch_TL3301NxxxxxG
Changed lines of the file:
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@@
 			)
 		)
-		(property "Footprint" "Button_Switch_THT:SW_PUSH_6mm_H9.5mm"
+		(property "Footprint" "Button_Switch_SMD:SW_Push_1P1T_NO_E-Switch_TL3301NxxxxxG"
 			(at 157.48 168.91 0)
 			(effects
