File: Project_Catronic/ProjetX.kicad_sch (KiCad schematic)
At the start: 4 parts

Commit message: Update KiCad project with latest schematic and PCB edits
Other:
- company: (none) -> ENSEA
- title: (none) -> CATRONIC
Changed lines of the file:
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@@
 	(generator_version "9.0")
 	(paper "A4")
+	(title_block
+		(title "CATRONIC")
+		(date "2025-10-13")
+		(company "ENSEA")
+		(comment 1 "HAJAR AIT ALLA")
+		(comment 2 "IKRAM AFIF")
+		(comment 3 "FAKHRI MENJLI")
+	)
 	(junction
 		(at 29.21 31.75)
